File: DRV8350S_Double/DRV8350S_Double.sch (KiCad schematic (older format))
At the start: 248 parts, among them IC1 MCP1501T-33, J1 USB_OTG, J10 Screw_Terminal_01x01, J11 Screw_Terminal_01x01, J12 Screw_Terminal_01x01, J13 Screw_Terminal_01x01, J14 Screw_Terminal_01x01, J15 Screw_Terminal_01x01, J16 Screw_Terminal_01x01, J17 Screw_Terminal_01x01, J18 Conn_01x08, J2 Conn_02x07_Odd_Even, J3 Conn_01x04, J4 47272-0001, J5 Conn_01x08, J6 Conn_01x08, J7 Conn_01x08, J8 Conn_01x08, J9 47272-0001, Q1 Q_NMOS_GDS, Q10 Q_NMOS_GDS, Q11 Q_NMOS_GDS, Q12 Q_NMOS_GDS, Q2 Q_NMOS_GDS, Q3 Q_NMOS_GDS, Q4 Q_NMOS_GDS, Q5 Q_NMOS_GDS, Q6 Q_NMOS_GDS, Q7 Q_NMOS_GDS, Q8 Q_NMOS_GDS, Q9 Q_NMOS_GDS, SW2 SW_Push, U1 LM5017MR, U10 SN65LVDS31D, U11 LM324DR, U12 LM324DR, U13 ESD122DMXR, U14 SN65LVDS33D, U15 LSF0204PWR, U16 LSF0204PWR, U17 LM324DR, U2 ADUM4160, U3 LM2576HVS-5, U4 LM2576HVS-3.3, U5 ISO1050-CUSTOM-SuperDriver_1.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, U6 STM32H743VITx, U7 DRV8350, U8 DRV8350, U9 SN65LVDS31D, Y1 SIT8008AI-82-33E-22.118400

Commit message: fixed iso_gnd miss
Parts:
- added JP5: SJ-O, Jumper:SolderJumper-2_P1.3mm_Open_TrianglePad1.0x1.5mm, symbol Jumper:SolderJumper_2_Open
- added NA3: Image, EVCONCEPT:qrcode_github, symbol Final_BLDC_Driver-rescue:Image-EV_Concept
Connections:
- net GND: now also JP5.2 (B)
- net GND_ISO: now also JP5.1 (A)
Other:
- moved on the sheet: JP4
Changed lines of the file:
@@
 L Jumper:SolderJumper_2_Open JP4
 U 1 1 648EBF91
-P 15000 12800
-F 0 "JP4" H 15000 13005 50  0000 C CNN
-F 1 "SJ-O" H 15000 12914 50  0000 C CNN
-F 2 "Jumper:SolderJumper-2_P1.3mm_Open_TrianglePad1.0x1.5mm" H 15000 12800 50  0001 C CNN
-F 3 "~" H 15000 12800 50  0001 C CNN
-	1    15000 12800
-	0    -1   -1   0
+P 15200 14700
+F 0 "JP4" H 15200 14905 50  0000 C CNN
+F 1 "SJ-O" H 15200 14814 50  0000 C CNN
+F 2 "Jumper:SolderJumper-2_P1.3mm_Open_TrianglePad1.0x1.5mm" H 15200 14700 50  0001 C CNN
+F 3 "~" H 15200 14700 50  0001 C CNN
+	1    15200 14700
+	1    0    0    -1
 $EndComp
 $Comp
 L power:+5V #PWR0176
 U 1 1 64A1159B
-P 15000 12650
-F 0 "#PWR0176" H 15000 12500 50  0001 C CNN
-F 1 "+5V" H 15015 12823 50  0000 C CNN
-F 2 "" H 15000 12650 50  0001 C CNN
-F 3 "" H 15000 12650 50  0001 C CNN
-	1    15000 12650
-	1    0    0    -1
-$EndComp
-Text GLabel 15000 12950 3    50   Input ~ 0
+P 15450 14600
+F 0 "#PWR0176" H 15450 14450 50  0001 C CNN
+F 1 "+5V" H 15465 14773 50  0000 C CNN
+F 2 "" H 15450 14600 50  0001 C CNN
+F 3 "" H 15450 14600 50  0001 C CNN
+	1    15450 14600
+	1    0    0    -1
+$EndComp
+Text GLabel 15050 14700 0    50   Input ~ 0
 5V_ISO
 $Comp
@@
 	1    0    0    -1
 $EndComp
+$Comp
+L Final_BLDC_Driver-rescue:Image-EV_Concept NA3
+U 1 1 61AAB7FC
+P 13800 20100
+F 0 "NA3" H 13978 20146 50  0000 L CNN
+F 1 "Image" H 13978 20055 50  0000 L CNN
+F 2 "EVCONCEPT:qrcode_github" H 13800 20100 50  0001 C CNN
+F 3 "" H 13800 20100 50  0001 C CNN
+	1    13800 20100
+	1    0    0    -1
+$EndComp
+$Comp
+L Jumper:SolderJumper_2_Open JP5
+U 1 1 61B35082
+P 15200 15000
+F 0 "JP5" H 15200 15205 50  0000 C CNN
+F 1 "SJ-O" H 15200 15114 50  0000 C CNN
+F 2 "Jumper:SolderJumper-2_P1.3mm_Open_TrianglePad1.0x1.5mm" H 15200 15000 50  0001 C CNN
+F 3 "~" H 15200 15000 50  0001 C CNN
+	1    15200 15000
+	1    0    0    -1
+$EndComp
+Text GLabel 15050 15000 0    50   Input ~ 0
+GND_ISO
+Wire Wire Line
+	15350 14700 15450 14700
+$Comp
+L power:GND #PWR0189
+U 1 1 6208B572
+P 15450 15100
+F 0 "#PWR0189" H 15450 14850 50  0001 C CNN
+F 1 "GND" H 15455 14927 50  0000 C CNN
+F 2 "" H 15450 15100 50  0001 C CNN
+F 3 "" H 15450 15100 50  0001 C CNN
+	1    15450 15100
+	1    0    0    -1
+$EndComp
+Wire Wire Line
+	15450 15100 15450 15000
+Wire Wire Line
+	15450 15000 15350 15000
+Wire Wire Line
+	15450 14600 15450 14700
 $EndSCHEMATC
