File: MA732_encoder/MA710_encoder.kicad_pcb (KiCad board)
At the start: 2 copper layers, 41 x 50.1 mm, 10 parts, among them J4 47272-0001, U1 MA730, U14 SN65LVDS33D, U9 SN65LVDS31D

Commit message: Commiting a ton of work, working current, position sensors, motion pos calibration routine done
Parts:
- added J1: Conn_01x02_Male, Connector_PinHeader_2.54mm:PinHeader_1x02_P2.54mm_Vertical, F.Cu at (152.7, 136.7)
- added R4: 0Ω, Resistor_SMD:R_0603_1608Metric, F.Cu at (170.1, 130.8)
Connections:
- J4 pad 1: SPI6_MISO_+ -> SPI6_nSS_-
- J4 pad 10: SPI6_nSS_+ -> SPI6_MISO_-
- J4 pad 12: SPI6_nSS_- -> SPI6_MISO_+
- J4 pad 13: (no net) -> TEMP_1
- J4 pad 14: (no net) -> unconnected-(J4-Pad14)
- J4 pad 15: (no net) -> +3V3
- J4 pad 16: (no net) -> +3V3
- J4 pad 17: (no net) -> +3V3
- J4 pad 18: (no net) -> unconnected-(J4-Pad18)
- J4 pad 3: SPI6_MISO_- -> SPI6_nSS_+
- J4 pad 4: SPI6_MOSI_+ -> SPI6_SCK_-
- J4 pad 6: SPI6_MOSI_- -> SPI6_SCK_+
- J4 pad 7: SPI6_SCK_+ -> SPI6_MOSI_-
- J4 pad 9: SPI6_SCK_- -> SPI6_MOSI_+
- U1 pad 1: (no net) -> unconnected-(U1-Pad1)
- U1 pad 11: (no net) -> unconnected-(U1-Pad11)
- U1 pad 14: (no net) -> unconnected-(U1-Pad14)
- U1 pad 15: (no net) -> unconnected-(U1-Pad15)
- U1 pad 16: (no net) -> unconnected-(U1-Pad16)
- U1 pad 2: (no net) -> unconnected-(U1-Pad2)
- U1 pad 3: (no net) -> unconnected-(U1-Pad3)
- U1 pad 6: (no net) -> unconnected-(U1-Pad6)
- U1 pad 9: (no net) -> unconnected-(U1-Pad9)
- U14 pad 13: (no net) -> unconnected-(U14-Pad13)
- U14 pad 14: (no net) -> unconnected-(U14-Pad14)
- U14 pad 15: (no net) -> unconnected-(U14-Pad15)
- U9 pad 10: (no net) -> unconnected-(U9-Pad10)
- U9 pad 11: (no net) -> unconnected-(U9-Pad11)
- U9 pad 13: (no net) -> unconnected-(U9-Pad13)
- U9 pad 14: (no net) -> unconnected-(U9-Pad14)
- U9 pad 15: (no net) -> unconnected-(U9-Pad15)
- U9 pad 5: (no net) -> unconnected-(U9-Pad5)
- U9 pad 6: (no net) -> unconnected-(U9-Pad6)
- U9 pad 7: (no net) -> unconnected-(U9-Pad7)
- U9 pad 9: (no net) -> unconnected-(U9-Pad9)
Routing:
- net TEMP_1: track 0.00 -> 21.7 mm, vias 0 -> 2
- net SPI6_MOSI_-: track 29.4 -> 44.6 mm, vias 0 -> 1
- net +3V3: track 29.3 -> 44.4 mm, vias 3 -> 4
- net SPI6_MOSI_+: track 30.9 -> 44.6 mm, vias 0 -> 1
- net SPI6_MISO_+: track 39.6 -> 32.3 mm, vias 0 -> 1
- net SPI6_MISO_-: track 38.4 -> 32.3 mm, vias 0 -> 1
- net SPI6_SCK_+: track 49.7 -> 43.9 mm
- net SPI6_nSS_+: track 44.6 -> 49.3 mm
- net SPI6_SCK_-: track 46.7 -> 42.9 mm
- net SPI6_nSS_-: track 46.1 -> 49.3 mm
Other:
- board text added: "DP Fixed Pos Sensor 2/14/2022 Logan Rosenmayer"
