File: HARDWARE/CURRENT_SENSE/Current_Sense.kicad_pcb (KiCad board)
At the start: 2 copper layers, 69.9 x 25.4 mm, 3 parts, among them J5 Conn_01x08, U1 HO-150-PW-0000

Commit message: Silk Screen Changes
Other:
- board size 69.9 x 25.4 mm -> 69.8 x 25.4 mm
- net class Default removed
- board text added: "MidwestMotorBoy Current Sense Rev 1.0 11/30/21"
- board text removed: "Logan Rosenmayer Current Sense Rev 1.0 11/30/21"
