File: HARDWARE/CURRENT_SENSE Tard version/Current_Sense.kicad_pcb (KiCad board)
At the start: 2 copper layers, 69.8 x 25.4 mm, 3 parts, among them J5 Conn_01x08, U1 HO-150-PW-0000

Commit message: Silk Screen Changes
Other:
- board text added: "MidwestMotorBoy Current Sense Tard Version (C1 ONLY)Rev 1.0 11/30/21"
- board text removed: "Logan Rosenmayer Current Sense Tard Version (C1 ONLY)Rev 1.0 11/30/21"
Changed lines of the file:
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@@
   (gr_arc (start 124.46 73.66) (mid 126.256051 74.403949) (end 127 76.2) (layer "Edge.Cuts") (width 0.05))
   (gr_arc (start 127 96.52) (mid 126.256051 98.316051) (end 124.46 99.06) (layer "Edge.Cuts") (width 0.05))
-  (gr_text "Logan Rosenmayer\nCurrent Sense Tard Version\n(C1 ONLY)Rev 1.0\n11/30/21" (at 115.697 95.758) (layer "F.SilkS")
+  (gr_text "MidwestMotorBoy\nCurrent Sense Tard Version\n(C1 ONLY)Rev 1.0\n11/30/21" (at 115.697 95.758) (layer "F.SilkS")
     (effects (font (size 1 1) (thickness 0.15)))
   )
