File: HARDWARE/DRV8350S_Double/DRV8350S_Double.kicad_pcb (KiCad board)
At the start: 4 copper layers, 180.5 x 154.9 mm, 252 parts, among them IC1 MCP1501T-33, J1 USB_OTG, J10 Screw_Terminal_01x01, J11 Screw_Terminal_01x01, J12 Screw_Terminal_01x01, J13 Screw_Terminal_01x01, J14 Screw_Terminal_01x01, J15 Screw_Terminal_01x01, J16 Screw_Terminal_01x01, J17 Screw_Terminal_01x01, J18 Conn_01x08, J2 Conn_02x07_Odd_Even, J3 Conn_01x04, J4 47272-0001, J5 Conn_01x08, J6 Conn_01x08, J7 Conn_01x08, J8 Conn_01x08, J9 47272-0001, Q1 Q_NMOS_GDS, Q10 Q_NMOS_GDS, Q11 Q_NMOS_GDS, Q12 Q_NMOS_GDS, Q2 Q_NMOS_GDS, Q3 Q_NMOS_GDS, Q4 Q_NMOS_GDS, Q5 Q_NMOS_GDS, Q6 Q_NMOS_GDS, Q7 Q_NMOS_GDS, Q8 Q_NMOS_GDS, Q9 Q_NMOS_GDS, SW2 SW_Push, U1 LM5017MR, U10 SN65LVDS31D, U11 LM324DR, U12 LM324DR, U14 SN65LVDS33D, U15 LSF0204PWR, U16 LSF0204PWR, U17 LM324DR, U18 USBLC6-2SC6, U2 ADUM4160, U3 LM2576HVS-5, U4 LM2576HVS-3.3, U5 ISO1050-CUSTOM-SuperDriver_1.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, U6 STM32H743VITx, U7 DRV8350, U8 DRV8350, U9 SN65LVDS31D, Y1 SIT8008AI-82-33E-22.118400

Commit message: Silk Screen Changes
Other:
- board text added: "MidwestMotorBoy Double DRV8350S 11/12/21 SEM REV 1.0"
- board text removed: "Logan Rosenmayer Double DRV8350S 11/12/21 SEM REV 1.0"
Changed lines of the file:
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@@
     (effects (font (size 5 5) (thickness 1)))
   )
-  (gr_text "Logan Rosenmayer\nDouble DRV8350S\n11/12/21\nSEM\nREV 1.0" (at 187.96 26.67) (layer "F.SilkS")
+  (gr_text "MidwestMotorBoy\nDouble DRV8350S\n11/12/21\nSEM\nREV 1.0" (at 187.96 26.67) (layer "F.SilkS")
     (effects (font (size 1.5 1.5) (thickness 0.3)))
   )
