File: HARDWARE/MA732_encoder/MA710_encoder.kicad_pcb (KiCad board)
At the start: 2 copper layers, 41 x 50.1 mm, 12 parts, among them J1 Conn_01x02_Male, J4 47272-0001, U1 MA730, U14 SN65LVDS33D, U9 SN65LVDS31D

Commit message: Silk Screen Changes
Other:
- board text added: "DP Fixed Pos Sensor 2/14/2022 MidwestMotorBoy"
- board text removed: "DP Fixed Pos Sensor 2/14/2022 Logan Rosenmayer"
Changed lines of the file:
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@@
   (gr_arc (start 179.068117 141.220674) (mid 164.568073 145.059744) (end 150.050501 141.287499) (layer "Edge.Cuts") (width 0.05))
   (gr_arc (start 150.079001 130.069999) (mid 164.394641 95.000269) (end 179.069999 129.920999) (layer "Edge.Cuts") (width 0.05))
-  (gr_text "DP Fixed Pos Sensor\n2/14/2022\nLogan Rosenmayer" (at 152.4 115.316 90) (layer "F.SilkS")
+  (gr_text "DP Fixed Pos Sensor\n2/14/2022\nMidwestMotorBoy" (at 152.4 115.316 90) (layer "F.SilkS")
     (effects (font (size 1 1) (thickness 0.15)))
   )
